File: kicad project/midea-ac-pen.kicad_pcb (KiCad board)
At the start: 2 copper layers, 50 x 24 mm, 8 parts, among them J1 Conn_01x04_Pin, Q1 2N3904, Q2 2N3904

Commit message: Fix library names and remove value field from ESP32 symbol
Parts:
- J1: footprint ESP32_C3_Super_Mini:PCB_USB -> Project Libraries:PCB_USB
- U1: footprint ESP32_C3_Super_Mini:ESP32_C3_Super_Mini -> Project Libraries:ESP32_C3_Super_Mini
Changed lines of the file:
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@@
 	(net 30 "unconnected-(U1-GPIO_8-Pad11)_1")
 	(net 31 "unconnected-(U1-GPIO_6-Pad9)_1")
-	(footprint "ESP32_C3_Super_Mini:PCB_USB"
+	(footprint "Project Libraries:PCB_USB"
 		(layer "F.Cu")
 		(at 89.6 117)
@@
 		(embedded_fonts no)
 	)
-	(footprint "ESP32_C3_Super_Mini:ESP32_C3_Super_Mini"
+	(footprint "Project Libraries:ESP32_C3_Super_Mini"
 		(layer "F.Cu")
 		(at 121.8 117 -90)
@@
 			(keep_text_aligned yes)
 		)
-		(gr_text "1.84"
+		(gr_text "1,84"
 			(at 143.65 128.08 90)
 			(layer "Edge.Cuts")
@@
 			(keep_text_aligned yes)
 		)
-		(gr_text "1.84"
+		(gr_text "1,84"
 			(at 143.85 105.92 90)
 			(layer "Edge.Cuts")

Commit message: Finish board design
Parts:
- added JP1: SolderJumper_2_Open, Jumper:SolderJumper-2_P1.3mm_Open_RoundedPad1.0x1.5mm, B.Cu at (102.5, 120.8)
- added JP2: SolderJumper_2_Bridged, Jumper:SolderJumper-2_P1.3mm_Bridged_RoundedPad1.0x1.5mm, B.Cu at (102.5, 118.2)
- added JP3: SolderJumper_2_Open, Jumper:SolderJumper-2_P1.3mm_Open_RoundedPad1.0x1.5mm, B.Cu at (102.5, 115.8)
- added JP4: SolderJumper_2_Bridged, Jumper:SolderJumper-2_P1.3mm_Bridged_RoundedPad1.0x1.5mm, B.Cu at (102.5, 113.2)
Connections:
- J1 pad 2: AC_RX -> D-
- J1 pad 3: AC_TX -> D+
Routing:
- net GND: track 0.00 -> 67.2 mm
- net 3.3V: track 0.00 -> 24.0 mm
- net D+: track 0.00 -> 17.4 mm, vias 0 -> 3
- net D-: track 0.00 -> 17.3 mm, vias 0 -> 1
- net AC_RX: track 23.3 -> 12.6 mm
- net ESP_RX: track 38.2 -> 41.5 mm
- net 5V: track 50.9 -> 48.0 mm
- net AC_TX: track 17.1 -> 14.3 mm
- net ESP_TX: track 14.4 -> 15.9 mm
Other:
- board size 50 x 24 mm -> 50 x 22.4 mm
